File: PCB/plus/musec_plus.kicad_pcb (KiCad board)
At the start: 2 copper layers, 308 x 193 mm, 61 parts, among them J1 Pedal, J2 PJ313, J3 PJ313, SW1 SW_DIP_x01, SW2 SW_DIP_x01, SW3 SW_DIP_x01, SW4 SW_DIP_x01, SW5 SW_DIP_x01, SW6 SW_DIP_x01, SW7 SW_DIP_x01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

Commit message: Musec Pico+ PCB v1.0
Parts:
- SW1, SW2, SW3, SW4, SW5: footprint musec_pico:SW_Kailh_Choc_V1V2_1.00u_LED -> musec_pico:Musec_ChocV1V2_x2_Combo
- moved C6 49.5 mm to (125.1, 65.6)
- moved C9 47.1 mm to (291.7, 202.3), turned to 0 degrees
- moved C8 25.8 mm to (205.4, 78.5), turned to 0 degrees
- moved C10 21.0 mm to (310.7, 84.3), turned to 0 degrees
- moved J1 6.73 mm to (114.2, 202.6)
- moved C7 0.82 mm to (138.8, 200.9)
Routing:
- net +5V: track 0.00 -> 1019.9 mm, vias 0 -> 13
- net /SCL: track 250.7 -> 893.0 mm, vias 5 -> 16
- net /SDA: track 286.9 -> 911.0 mm, vias 5 -> 15
- net Net-(J2-T): track 0.00 -> 495.4 mm, vias 0 -> 2
- net /K4: track 0.00 -> 262.7 mm, vias 0 -> 2
- net /VB5: track 52.2 -> 288.2 mm, vias 1 -> 5
- net /K5: track 0.00 -> 231.7 mm, vias 0 -> 2
- net Net-(D21-Out): track 0.00 -> 201.1 mm
- net /VB4: track 52.2 -> 245.1 mm, vias 1 -> 5
- net /K2: track 0.00 -> 179.4 mm, vias 0 -> 2
- net /K7: track 0.00 -> 162.7 mm
- net Net-(J1-Pin_2): track 0.00 -> 161.5 mm, vias 0 -> 1
- net Net-(J1-Pin_3): track 0.00 -> 157.9 mm, vias 0 -> 1
- net /K3: track 0.00 -> 142.2 mm
- net /VB3: track 52.2 -> 189.0 mm, vias 1 -> 5
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- added copper zone on B.Cu, net GND
- added copper zone on F.Cu, net GND
Other:
- board size 308 x 193 mm -> 308 x 170 mm

Commit message: Musec Pico+ PCB v1.01
Parts:
- moved C7 11.7 mm to (150.6, 200.9), turned to 0 degrees
Routing:
- net +5V: track 1019.9 -> 1021.3 mm, vias 13 -> 14
Other:
- outline, holes or cut-outs redrawn
- board text added: "v1.01"
- board text removed: "v1.0"

Commit message: Explicit I2C Pull-ups
Parts:
- added R3: 5K1, Resistor_SMD:R_0603_1608Metric_Pad0.98x0.95mm_HandSolder, F.Cu at (174.4, 77.1)
- added R4: 5K1, Resistor_SMD:R_0603_1608Metric_Pad0.98x0.95mm_HandSolder, F.Cu at (174.4, 74.7)
Routing:
- net /SDA: track 911.0 -> 929.0 mm, vias 15 -> 16
- net /SCL: track 893.0 -> 908.1 mm, vias 16 -> 17
- net +3V3: track 0.00 -> 10.9 mm, vias 0 -> 1
- net /K4: track 262.7 -> 271.7 mm
- net +5V: track 1021.3 -> 1020.4 mm
- net GND: vias 48 -> 51
Other:
- board text added: "Musec Pico+ v1.1"
- board text added: "github.com/whowechina"
- board text removed: "Musec Pico+"
- board text removed: "v1.01"
