File: PCB/plus/musec_plus.kicad_pcb (KiCad board)
At the start: 2 copper layers, 308 x 170 mm, 63 parts, among them J1 Pedal, J2 PJ313, J3 PJ313, SW1 SW_DIP_x01, SW2 SW_DIP_x01, SW3 SW_DIP_x01, SW4 SW_DIP_x01, SW5 SW_DIP_x01, SW6 SW_DIP_x01, SW7 SW_DIP_x01, U1 PiPico, U3 TMAG5273, U4 TMAG5273, U5 TMAG5273, U6 TMAG5273, U7 TMAG5273

Commit message: PCB V1.2, add pedal TRS ring option
Connections:
- J2 pad 2: GND -> Net-(J2-R)
- J3 pad 2: GND -> Net-(J2-R)
- U1 pad 6: unconnected-(U1-GPIO4-Pad6) -> Net-(J2-R)
Routing:
- net Net-(J2-R): track 0.00 -> 501.0 mm, vias 0 -> 2
- net Net-(J2-T): track 495.4 -> 497.2 mm
- net Net-(J1-Pin_2): track 161.5 -> 160.5 mm
- net Net-(D1-In): track 76.1 -> 75.3 mm
- net GND: vias 51 -> 55
Other:
- board text added: "Musec Pico+ v1.2"
- board text removed: "Musec Pico+ v1.1"
