File: PCB/plus/musec_plus.kicad_sch (KiCad schematic)
At the start: 61 parts, among them J1 Pedal, J2 PJ313, J3 PJ313, SW1 SW_DIP_x01, SW2 SW_DIP_x01, SW3 SW_DIP_x01, SW4 SW_DIP_x01, SW5 SW_DIP_x01, SW6 SW_DIP_x01, SW7 SW_DIP_x01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

Commit message: Musec Pico+ PCB v1.0
Parts:
- SW1, SW2, SW3, SW4, SW5: footprint musec_pico:SW_Kailh_Choc_V1V2_1.00u_LED -> musec_pico:Musec_ChocV1V2_x2_Combo
Changed lines of the file:
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@@
 			)
 		)
-		(property "Footprint" "musec_pico:SW_Kailh_Choc_V1V2_1.00u_LED"
+		(property "Footprint" "musec_pico:Musec_ChocV1V2_x2_Combo"
 			(at 203.2 125.73 0)
 			(effects
@@
 			)
 		)
-		(property "Footprint" "musec_pico:SW_Kailh_Choc_V1V2_1.00u_LED"
+		(property "Footprint" "musec_pico:Musec_ChocV1V2_x2_Combo"
 			(at 190.5 140.97 0)
 			(effects
@@
 			)
 		)
-		(property "Footprint" "musec_pico:SW_Kailh_Choc_V1V2_1.00u_LED"
+		(property "Footprint" "musec_pico:Musec_ChocV1V2_x2_Combo"
 			(at 177.8 125.73 0)
 			(effects
@@
 			)
 		)
-		(property "Footprint" "musec_pico:SW_Kailh_Choc_V1V2_1.00u_LED"
+		(property "Footprint" "musec_pico:Musec_ChocV1V2_x2_Combo"
 			(at 216.535 140.97 0)
 			(effects
@@
 			)
 		)
-		(property "Footprint" "musec_pico:SW_Kailh_Choc_V1V2_1.00u_LED"
+		(property "Footprint" "musec_pico:Musec_ChocV1V2_x2_Combo"
 			(at 229.235 125.73 0)
 			(effects

Commit message: Explicit I2C Pull-ups
Parts:
- added R3, R4: 5K1, Resistor_SMD:R_0603_1608Metric_Pad0.98x0.95mm_HandSolder, symbol Device:R_Small
Connections:
- net +3V3: now also R3.2, R4.2
- net SCL: now also R3.1
- net SDA: now also R4.1
